File: UPDI-Programmer/USB-C-UPDI.brd (EAGLE design)
At the start: 27.4 x 18.3 mm, 9 parts, among them IC1 FT232RL, J2 61300511121

Commit message: Add files via upload
Routing:
- net GND: track 75.1 -> 77.7 mm
- net N$5: track 27.5 -> 29.2 mm
- net N$13: track 16.3 -> 17.1 mm
- net N$1: track 4.57 -> 5.16 mm
