File: USB-C UPDI/USB-C-UPDI.brd (EAGLE design)
At the start: 27.4 x 18.3 mm, 9 parts, among them IC1 FT232RL, J2 61300511121

Commit message: Updates
Parts:
- moved C10 0.10 mm to (5.62, 5.41)
Routing:
- net GND: track 77.7 -> 78.6 mm
- net RX: track 24.8 -> 25.7 mm
