File: USB-C UPDI/ftdi2updi.brd (EAGLE design)
At the start: 33.1 x 26.6 mm, 6 parts, among them J2 61300511121

Commit message: updates
Parts:
- moved U$1 3.15 mm to (31.1, 19.9)
Connections:
- net N$1: no longer U$1.4
- net N$2: no longer U$1.5
Routing:
- net N$2: track 26.9 -> 29.9 mm
- net N$1: track 26.7 -> 28.7 mm
- net GND: track 32.9 -> 31.9 mm
- net VCC: track 19.0 -> 19.6 mm
Changed lines of the file:
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@@
 <setting verticaltext="up"/>
 </settings>
-<grid distance="0.1" unitdist="mm" unit="mm" style="lines" multiple="1" display="yes" altdistance="5" altunitdist="mil" altunit="mil"/>
+<grid distance="0.1" unitdist="mm" unit="mm" style="lines" multiple="1" display="no" altdistance="5" altunitdist="mil" altunit="mil"/>
 <layers>
 <layer number="1" name="Top" color="4" fill="1" visible="yes" active="yes"/>
@@
 <attribute name="VALUE" x="5.031621875" y="6.911959375" size="0.6096" layer="28" font="vector" ratio="20" rot="MR90" align="top-center"/>
 </element>
-<element name="U$1" library="fab_new" package="1X06SMD" value="CONN_06_FTDI-SMD-HEADER" x="27.901621875" y="19.891959375" smashed="yes" rot="MR0">
-<attribute name="NAME" x="29.806621875" y="16.716959375" size="1.27" layer="26" rot="MR90"/>
+<element name="U$1" library="fab_new" package="1X06SMD" value="CONN_06_FTDI-SMD-HEADER" x="31.051621875" y="19.891959375" smashed="yes" rot="MR0">
+<attribute name="NAME" x="32.956621875" y="16.716959375" size="1.27" layer="26" rot="MR90"/>
 </element>
 </elements>
@@
 <signal name="VCC">
 <contactref element="U$1" pad="3"/>
-<wire x1="29.675221875" y1="21.161959375" x2="30.966421875" y2="19.870759375" width="0.4572" layer="16"/>
-<wire x1="27.901621875" y1="21.161959375" x2="29.675221875" y2="21.161959375" width="0.4572" layer="16"/>
-<wire x1="30.966421875" y1="10.4403" x2="28.5723" y2="8.046178125" width="0.4572" layer="16"/>
+<wire x1="31.051621875" y1="21.161959375" x2="32.851621875" y2="21.161959375" width="0.4572" layer="16"/>
+<wire x1="33.166421875" y1="20.847159375" x2="32.851621875" y2="21.161959375" width="0.4572" layer="16"/>
+<wire x1="33.166421875" y1="20.847159375" x2="33.166421875" y2="12.6403" width="0.4572" layer="16"/>
+<wire x1="33.166421875" y1="12.6403" x2="28.5723" y2="8.046178125" width="0.4572" layer="16"/>
 <wire x1="28.5723" y1="8.046178125" x2="28.5723" y2="5.424303125" width="0.4572" layer="16"/>
-<wire x1="30.966421875" y1="19.870759375" x2="30.966421875" y2="10.4403" width="0.4572" layer="16"/>
 </signal>
 <signal name="GND">
 <contactref element="U$1" pad="1"/>
-<wire x1="27.901621875" y1="26.241959375" x2="30.821621875" y2="26.241959375" width="0.4572" layer="16"/>
 <wire x1="26.70118125" y1="3.801959375" x2="26.024040625" y2="4.4791" width="0.4572" layer="16"/>
 <wire x1="26.024040625" y1="4.4791" x2="26.024040625" y2="5.489440625" width="0.4572" layer="16"/>
-<wire x1="30.821621875" y1="26.241959375" x2="32.581621875" y2="24.481959375" width="0.4572" layer="16"/>
-<wire x1="32.581621875" y1="24.481959375" x2="32.581621875" y2="5.501959375" width="0.4572" layer="16"/>
-<wire x1="32.581621875" y1="5.501959375" x2="30.881621875" y2="3.801959375" width="0.4572" layer="16"/>
-<wire x1="30.881621875" y1="3.801959375" x2="26.70118125" y2="3.801959375" width="0.4572" layer="16"/>
+<wire x1="34.081621875" y1="25.281959375" x2="33.121621875" y2="26.241959375" width="0.4572" layer="16"/>
+<wire x1="31.051621875" y1="26.241959375" x2="33.121621875" y2="26.241959375" width="0.4572" layer="16"/>
+<wire x1="34.081621875" y1="25.281959375" x2="34.081621875" y2="7.901959375" width="0.4572" layer="16"/>
+<wire x1="34.081621875" y1="7.901959375" x2="29.981621875" y2="3.801959375" width="0.4572" layer="16"/>
+<wire x1="29.981621875" y1="3.801959375" x2="26.70118125" y2="3.801959375" width="0.4572" layer="16"/>
 </signal>
 <signal name="N$1">
-<contactref element="U$1" pad="4"/>
 <contactref element="S1" pad="2"/>
 <wire x1="8.841621875" y1="9.736959375" x2="9.904571875" y2="10.799909375" width="0.4572" layer="16"/>
-<wire x1="24.679571875" y1="10.799909375" x2="25.081621875" y2="11.201959375" width="0.4572" layer="16"/>
-<wire x1="25.081621875" y1="11.201959375" x2="25.081621875" y2="17.901959375" width="0.4572" layer="16"/>
-<wire x1="25.081621875" y1="17.901959375" x2="25.801621875" y2="18.621959375" width="0.4572" layer="16"/>
-<wire x1="25.801621875" y1="18.621959375" x2="27.901621875" y2="18.621959375" width="0.4572" layer="16"/>
-<wire x1="9.904571875" y1="10.799909375" x2="24.679571875" y2="10.799909375" width="0.4572" layer="16"/>
+<wire x1="9.904571875" y1="10.799909375" x2="25.079571875" y2="10.799909375" width="0.4572" layer="16"/>
+<wire x1="26.2" y1="11.9203375" x2="26.2" y2="16.7" width="0.4572" layer="16"/>
+<wire x1="26.2" y1="16.7" x2="28.1" y2="18.6" width="0.4572" layer="16"/>
+<wire x1="28.1" y1="18.6" x2="31.1" y2="18.6" width="0.4572" layer="16"/>
+<wire x1="25.079571875" y1="10.799909375" x2="26.2" y2="11.9203375" width="0.4572" layer="16"/>
 </signal>
 <signal name="N$2">
-<contactref element="U$1" pad="5"/>
 <contactref element="S1" pad="5"/>
 <wire x1="9.530421875" y1="4.149959375" x2="8.920821875" y2="4.149959375" width="0.4572" layer="16"/>
@@
 <wire x1="16.912821875" y1="8.217159375" x2="14.260021875" y2="5.564359375" width="0.4572" layer="1"/>
 <wire x1="23.646421875" y1="8.217159375" x2="16.912821875" y2="8.217159375" width="0.4572" layer="1"/>
-<wire x1="25.989621875" y1="10.560359375" x2="23.646421875" y2="8.217159375" width="0.4572" layer="16"/>
-<wire x1="25.989621875" y1="15.408359375" x2="25.989621875" y2="10.560359375" width="0.4572" layer="16"/>
-<wire x1="26.663221875" y1="16.081959375" x2="25.989621875" y2="15.408359375" width="0.4572" layer="16"/>
 <wire x1="8.920821875" y1="4.149959375" x2="8.841621875" y2="4.086959375" width="0.4572" layer="16"/>
-<wire x1="26.663221875" y1="16.081959375" x2="27.901621875" y2="16.081959375" width="0.4572" layer="16"/>
 <via x="13.383221875" y="5.564359375" extent="1-16" drill="0.6"/>
 <via x="23.646421875" y="8.217159375" extent="1-16" drill="0.6"/>
+<wire x1="29.2" y1="16.1" x2="31.400625" y2="16.1" width="0.4572" layer="16"/>
+<wire x1="27.9" y1="10.7707375" x2="25.346421875" y2="8.217159375" width="0.4572" layer="16"/>
+<wire x1="23.646421875" y1="8.217159375" x2="25.346421875" y2="8.217159375" width="0.4572" layer="16"/>
+<wire x1="27.9" y1="10.7707375" x2="27.9" y2="14.8" width="0.4572" layer="16"/>
+<wire x1="27.9" y1="14.8" x2="29.2" y2="16.1" width="0.4572" layer="16"/>
 </signal>
 <signal name="N$17">

Commit message: via updates
Routing:
- net S$1: track 0.00 -> 29.1 mm
Changed lines of the file:
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@@
 <wire x1="1.61928125" y1="11.352009375" x2="1.61928125" y2="4.479678125" width="0.015" layer="20"/>
 <wire x1="1.61928125" y1="4.479678125" x2="3.61928125" y2="2.479678125" width="0.015" layer="20" curve="90"/>
-<wire x1="3.61928125" y1="2.479678125" x2="32.753703125" y2="2.479678125" width="0.015" layer="20"/>
 <wire x1="32.753703125" y1="2.479678125" x2="34.753703125" y2="4.479678125" width="0.015" layer="20" curve="90"/>
 <wire x1="34.753703125" y1="4.479678125" x2="34.753703125" y2="27.072378125" width="0.015" layer="20"/>
@@
 <elements>
 <element name="D1" library="eagle_fab" package="MINI-SMA" value="SCHOTTKY" x="27.931621875" y="19.851959375" smashed="yes" rot="R225">
-<attribute name="NAME" x="30.625703125" y="20.749978125" size="1.27" layer="25" rot="R225"/>
 <attribute name="VALUE" x="27.931621875" y="23.444059375" size="1.27" layer="27" rot="R225"/>
 </element>
@@
 <attribute name="MANUFACTURER" value="Wurth Electronics Inc." x="45.036740625" y="-13.458040625" size="1.778" layer="27" display="off"/>
 <attribute name="MPN" value="61300511121" x="45.036740625" y="-13.458040625" size="1.778" layer="27" display="off"/>
-<attribute name="NAME" x="20.450740625" y="8.611959375" size="1.27" layer="25"/>
 <attribute name="VALUE" x="20.196740625" y="1.829959375" size="1.27" layer="27"/>
 </element>
 <element name="R1" library="eagle_fab" package="R1206FAB" value="1.5k" x="27.881621875" y="25.591959375" smashed="yes" rot="R225">
-<attribute name="NAME" x="30.036884375" y="25.951171875" size="1.016" layer="25" ratio="15" rot="R225"/>
 <attribute name="VALUE" x="27.5224125" y="28.46564375" size="1.016" layer="27" ratio="15" rot="R225"/>
 </element>
 <element name="R2" library="01_SparkFun" package="1206" value="470" x="27.801621875" y="14.581959375" smashed="yes" rot="R45">
-<attribute name="NAME" x="26.095371875" y="14.49215625" size="0.4064" layer="25" rot="R45"/>
 <attribute name="VALUE" x="27.891421875" y="12.5165" size="0.4064" layer="27" rot="R45"/>
 </element>
 <element name="S1" library="SparkFun-Switches" package="SWITCH_DPDT_SMD_AYZ0202" value="" x="8.841621875" y="6.911959375" smashed="yes" rot="MR0">
-<attribute name="NAME" x="12.651621875" y="6.911959375" size="0.6096" layer="26" font="vector" ratio="20" rot="MR90" align="bottom-center"/>
 <attribute name="PROD_ID" value="SWCH-08179" x="-7.668378125" y="-21.028040625" size="1.778" layer="28" rot="MR0" display="off"/>
 <attribute name="SF_SKU" value="COM-00597" x="-7.668378125" y="-21.028040625" size="1.778" layer="28" rot="MR0" display="off"/>
 <attribute name="VALUE" x="5.031621875" y="6.911959375" size="0.6096" layer="28" font="vector" ratio="20" rot="MR90" align="top-center"/>
 </element>
-<element name="U$1" library="fab_new" package="1X06SMD" value="CONN_06_FTDI-SMD-HEADER" x="31.051621875" y="19.891959375" smashed="yes" rot="MR0">
-<attribute name="NAME" x="32.956621875" y="16.716959375" size="1.27" layer="26" rot="MR90"/>
-</element>
+<element name="U$1" library="fab_new" package="1X06SMD" value="CONN_06_FTDI-SMD-HEADER" x="31.051621875" y="19.891959375" smashed="yes" rot="MR0"/>
 </elements>
 <signals>
@@
 <wire x1="25.694421875" y1="17.330459375" x2="26.76489375" y2="18.68523125" width="0.4572" layer="1"/>
 <wire x1="26.599221875" y1="13.598759375" x2="26.811671875" y2="13.592009375" width="0.4572" layer="1"/>
-<via x="3.463221875" y="3.826759375" extent="1-16" drill="0.6"/>
+<via x="3.463221875" y="3.826759375" extent="1-16" drill="0.6" diameter="1.3"/>
 </signal>
 <signal name="UPDI">
@@
 <wire x1="7.092021875" y1="9.636359375" x2="6.482421875" y2="9.636359375" width="0.4572" layer="16"/>
 <wire x1="8.506421875" y1="8.221959375" x2="7.092021875" y2="9.636359375" width="0.4572" layer="16"/>
-<wire x1="13.383221875" y1="8.721959375" x2="12.883221875" y2="8.221959375" width="0.4572" layer="16"/>
-<wire x1="12.883221875" y1="8.221959375" x2="8.506421875" y2="8.221959375" width="0.4572" layer="16"/>
-<wire x1="26.475221875" y1="9.331559375" x2="13.992821875" y2="9.331559375" width="0.4572" layer="1"/>
-<wire x1="13.992821875" y1="9.331559375" x2="13.383221875" y2="8.721959375" width="0.4572" layer="1"/>
+<wire x1="13.383221875" y1="8.521959375" x2="13.083221875" y2="8.221959375" width="0.4572" layer="16"/>
+<wire x1="13.083221875" y1="8.221959375" x2="8.506421875" y2="8.221959375" width="0.4572" layer="16"/>
+<wire x1="26.475221875" y1="9.331559375" x2="14.192821875" y2="9.331559375" width="0.4572" layer="1"/>
+<wire x1="14.192821875" y1="9.331559375" x2="13.383221875" y2="8.521959375" width="0.4572" layer="1"/>
 <wire x1="28.428021875" y1="11.284359375" x2="26.475221875" y2="9.331559375" width="0.4572" layer="1"/>
 <wire x1="28.428021875" y1="14.008359375" x2="28.428021875" y2="11.284359375" width="0.4572" layer="1"/>
@@
 <wire x1="6.482421875" y1="9.636359375" x2="6.341621875" y2="9.736959375" width="0.1524" layer="16"/>
 <wire x1="26.904021875" y1="24.266759375" x2="26.7141875" y2="24.424525" width="0.2032" layer="1"/>
-<via x="13.383221875" y="8.721959375" extent="1-16" drill="0.6"/>
+<via x="13.383221875" y="8.521959375" extent="1-16" drill="0.6" diameter="1.3"/>
 </signal>
 <signal name="RX">
 <contactref element="S1" pad="4"/>
 <contactref element="J2" pad="1"/>
-<wire x1="15.749390625" y1="3.845159375" x2="11.359221875" y2="3.845159375" width="0.4572" layer="16"/>
+<wire x1="15.8969125" y1="3.845159375" x2="11.359221875" y2="3.845159375" width="0.4572" layer="16"/>
 <wire x1="11.359221875" y1="3.845159375" x2="11.341621875" y2="4.086959375" width="0.4572" layer="16"/>
-<wire x1="16.57951875" y1="5.591959375" x2="18.366740625" y2="5.591959375" width="0.4572" layer="16"/>
-<wire x1="16.57951875" y1="5.591959375" x2="15.749390625" y2="3.845159375" width="0.4572" layer="16"/>
+<wire x1="16.727040625" y1="5.591959375" x2="18.366740625" y2="5.591959375" width="0.4572" layer="16"/>
+<wire x1="16.727040625" y1="5.591959375" x2="15.8969125" y2="3.845159375" width="0.4572" layer="16"/>
 </signal>
 <signal name="TX">
@@
 <wire x1="14.260021875" y1="5.564359375" x2="13.383221875" y2="5.564359375" width="0.4572" layer="1"/>
 <wire x1="16.912821875" y1="8.217159375" x2="14.260021875" y2="5.564359375" width="0.4572" layer="1"/>
-<wire x1="23.646421875" y1="8.217159375" x2="16.912821875" y2="8.217159375" width="0.4572" layer="1"/>
+<wire x1="22.746421875" y1="8.217159375" x2="16.912821875" y2="8.217159375" width="0.4572" layer="1"/>
 <wire x1="8.920821875" y1="4.149959375" x2="8.841621875" y2="4.086959375" width="0.4572" layer="16"/>
-<via x="13.383221875" y="5.564359375" extent="1-16" drill="0.6"/>
-<via x="23.646421875" y="8.217159375" extent="1-16" drill="0.6"/>
+<via x="13.383221875" y="5.564359375" extent="1-16" drill="0.6" diameter="1.3"/>
+<via x="22.746421875" y="8.217159375" extent="1-16" drill="0.6" diameter="1.2"/>
 <wire x1="29.2" y1="16.1" x2="31.400625" y2="16.1" width="0.4572" layer="16"/>
 <wire x1="27.9" y1="10.7707375" x2="25.346421875" y2="8.217159375" width="0.4572" layer="16"/>
-<wire x1="23.646421875" y1="8.217159375" x2="25.346421875" y2="8.217159375" width="0.4572" layer="16"/>
+<wire x1="22.746421875" y1="8.217159375" x2="25.346421875" y2="8.217159375" width="0.4572" layer="16"/>
 <wire x1="27.9" y1="10.7707375" x2="27.9" y2="14.8" width="0.4572" layer="16"/>
 <wire x1="27.9" y1="14.8" x2="29.2" y2="16.1" width="0.4572" layer="16"/>
@@
 <wire x1="30.9271125" y1="27.25770625" x2="30.9445125" y2="27.488528125" width="0.2032" layer="1"/>
 </signal>
+<signal name="S$1">
+<wire x1="3.61928125" y1="2.479678125" x2="32.753703125" y2="2.479678125" width="0.015" layer="1"/>
+</signal>
 </signals>

Commit message: updates
Parts:
- moved D1 1.58 mm to (27.0, 18.6)
- moved S1 1.58 mm to (7.94, 5.61)
- moved R2 1.58 mm to (26.9, 13.3)
- moved U$1 1.58 mm to (30.2, 18.6)
- moved J2 1.58 mm to (22.5, 4.29)
- moved R1 1.58 mm to (27.0, 24.3)
Routing:
- net S$1: track 29.1 -> 0.00 mm

Commit message: updates
Routing:
- net RX: track 8.35 -> 9.14 mm
- net N$3: track 37.5 -> 36.7 mm

Commit message: updates
Parts:
- removed R1: 1.5k, eagle_fab:R1206FAB
- moved D1 3.45 mm to (27.6, 22.0)
- moved R2 1.99 mm to (27.5, 15.2)
- moved U$1 0.63 mm to (30.8, 18.8)
- moved S1 0.63 mm to (8.54, 5.81)
- moved J2 0.63 mm to (23.1, 4.49)
Connections:
- net GND renamed S$1
- removed net N$4: D1.KATHODE, R1.1
- removed net VCC: U$1.3
- new net S$3: D1.KATHODE
- net N$11: no longer R1.2
Routing:
- net S$1: track 31.9 -> 0.14 mm
- net GND: track 0.00 -> 11.1 mm
- net N$2: track 30.0 -> 41.1 mm
- net N$4: track 5.75 -> 0.00 mm
- net N$3: track 36.7 -> 39.9 mm
- net N$1: track 28.7 -> 31.2 mm
- net UPDI: track 14.4 -> 16.1 mm
- net VCC: track 19.6 -> 18.0 mm
- net N$11: track 39.2 -> 38.5 mm
