File: USB-C UPDI/ftdi2updi.sch (EAGLE design)
At the start: 6 parts, among them J2 61300511121

Commit message: updates
Parts:
- removed R1: 1.5k, eagle_fab:R1206FAB
Connections:
- removed net N$11: R1.2, S1.3
- net N$4: now also S1.3; no longer R1.1
Changed lines of the file:
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@@
 <part name="J2" library="Headers" library_urn="urn:adsk.eagle:library:11687645" deviceset="61300511121" device="" package3d_urn="urn:adsk.eagle:package:11390687/2"/>
 <part name="S1" library="SparkFun-Switches" deviceset="SWITCH-DPDT" device="-SMD-AYZ0202"/>
-<part name="R1" library="eagle_fab" deviceset="R" device="1206FAB" value="1.5k"/>
 <part name="U$1" library="fab_new" deviceset="CONN_06_FTDI-SMD-HEADER" device=""/>
 </parts>
@@
 <attribute name="NAME" x="48.26" y="37.846" size="1.778" layer="95" font="vector" rot="R180" align="bottom-center"/>
 <attribute name="VALUE" x="48.26" y="56.134" size="1.778" layer="96" font="vector" rot="R180" align="top-center"/>
-</instance>
-<instance part="R1" gate="G$1" x="33.02" y="40.64" smashed="yes">
-<attribute name="NAME" x="29.21" y="42.1386" size="1.778" layer="95"/>
-<attribute name="VALUE" x="29.21" y="37.338" size="1.778" layer="96"/>
 </instance>
 <instance part="U$1" gate="G$1" x="20.32" y="25.4" smashed="yes" rot="R270"/>
@@
 </segment>
 </net>
-<net name="N$11" class="0">
-<segment>
-<pinref part="S1" gate="G$1" pin="3"/>
-<wire x1="43.18" y1="40.64" x2="38.1" y2="40.64" width="0.1524" layer="91"/>
-<pinref part="R1" gate="G$1" pin="2"/>
-</segment>
-</net>
 <net name="RX" class="0">
 <segment>
@@
 <pinref part="D1" gate="G$1" pin="KATHODE"/>
 <wire x1="27.94" y1="50.8" x2="25.4" y2="50.8" width="0.1524" layer="91"/>
-<wire x1="27.94" y1="40.64" x2="25.4" y2="40.64" width="0.1524" layer="91"/>
 <wire x1="25.4" y1="40.64" x2="25.4" y2="50.8" width="0.1524" layer="91"/>
-<pinref part="R1" gate="G$1" pin="1"/>
+<pinref part="S1" gate="G$1" pin="3"/>
+<wire x1="25.4" y1="40.64" x2="43.18" y2="40.64" width="0.1524" layer="91"/>
 </segment>
 </net>
