File: USB-C UPDI/ftdi2updiCOPPER.brd (EAGLE design)
At the start: 33.1 x 26.6 mm, 5 parts, among them J2 61300511121

Commit message: gerber files
Parts:
- moved U$1 0.45 mm to (31.2, 18.8)
Routing:
- net VCC: track 18.0 -> 17.0 mm
Other:
- board text added: "470 Ω"
- board text added: "SCHOTTKY"
Changed lines of the file:
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@@
 <text x="20" y="6.1" size="0.7" layer="25">TX</text>
 <text x="17.4" y="6.1" size="0.7" layer="25">RX</text>
+<text x="25.5" y="21.4" size="0.5" layer="25" rot="R45">SCHOTTKY</text>
+<text x="27.2" y="16.4" size="0.5" layer="25" rot="R45">470 Ω</text>
 </plain>
 <attributes>
@@
 <attribute name="VALUE" x="4.731621875" y="5.811959375" size="0.6096" layer="28" font="vector" ratio="20" rot="MR90" align="top-center"/>
 </element>
-<element name="U$1" library="fab_new" package="1X06SMD" value="CONN_06_FTDI-SMD-HEADER" x="30.751621875" y="18.791959375" smashed="yes" rot="MR0"/>
+<element name="U$1" library="fab_new" package="1X06SMD" value="CONN_06_FTDI-SMD-HEADER" x="31.201621875" y="18.791959375" smashed="yes" rot="MR0"/>
 </elements>
 <signals>
@@
 <wire x1="26.299221875" y1="13.893959375" x2="26.299221875" y2="10.669959375" width="0.4572" layer="1"/>
 <wire x1="26.299221875" y1="13.893959375" x2="26.511671875" y2="14.192009375" width="0.4572" layer="1"/>
-<wire x1="25.394421875" y1="15.103559375" x2="25.394421875" y2="19.430459375" width="0.4572" layer="1"/>
-<wire x1="26.299221875" y1="14.198759375" x2="25.394421875" y2="15.103559375" width="0.4572" layer="1"/>
-<wire x1="25.394421875" y1="19.430459375" x2="26.46489375" y2="20.78523125" width="0.4572" layer="1"/>
+<wire x1="25.294421875" y1="15.203559375" x2="25.294421875" y2="19.3039" width="0.4572" layer="1"/>
+<wire x1="26.299221875" y1="14.198759375" x2="25.294421875" y2="15.203559375" width="0.4572" layer="1"/>
+<wire x1="25.294421875" y1="19.3039" x2="26.46489375" y2="20.78523125" width="0.4572" layer="1"/>
 <wire x1="26.299221875" y1="14.198759375" x2="26.511671875" y2="14.192009375" width="0.4572" layer="1"/>
 <via x="3.363221875" y="3.026759375" extent="1-16" drill="0.85" diameter="1.8"/>
@@
 <wire x1="28.128021875" y1="10.184359375" x2="26.475221875" y2="8.531559375" width="0.4572" layer="1"/>
 <wire x1="28.128021875" y1="14.608359375" x2="28.128021875" y2="10.184359375" width="0.4572" layer="1"/>
-<wire x1="26.704021875" y1="16.032359375" x2="28.128021875" y2="14.608359375" width="0.4572" layer="1"/>
-<wire x1="26.704021875" y1="16.032359375" x2="26.704021875" y2="17.846759375" width="0.4572" layer="1"/>
+<wire x1="26.404021875" y1="16.332359375" x2="28.128021875" y2="14.608359375" width="0.4572" layer="1"/>
+<wire x1="26.404021875" y1="16.332359375" x2="26.404021875" y2="17.546759375" width="0.4572" layer="1"/>
 <wire x1="6.182421875" y1="8.536359375" x2="6.041621875" y2="8.636959375" width="0.1524" layer="16"/>
 <via x="13.683221875" y="6.921959375" extent="1-16" drill="0.85" diameter="1.8"/>
 <wire x1="28.9" y1="20.0427375" x2="28.9" y2="23" width="0.4572" layer="1"/>
-<wire x1="26.704021875" y1="17.846759375" x2="28.9" y2="20.0427375" width="0.4572" layer="1"/>
+<wire x1="26.404021875" y1="17.546759375" x2="28.9" y2="20.0427375" width="0.4572" layer="1"/>
 </signal>
 <signal name="RX">
@@
 </signal>
 <signal name="VCC">
-<wire x1="33.166421875" y1="11.2403" x2="33.166421875" y2="16.747159375" width="0.4572" layer="16"/>
-<wire x1="33.166421875" y1="11.2403" x2="28.2723" y2="6.346178125" width="0.4572" layer="16"/>
+<wire x1="33.366421875" y1="11.4403" x2="33.366421875" y2="16.547159375" width="0.4572" layer="16"/>
+<wire x1="33.366421875" y1="11.4403" x2="28.2723" y2="6.346178125" width="0.4572" layer="16"/>
 <wire x1="28.2723" y1="6.346178125" x2="28.2723" y2="4.324303125" width="0.4572" layer="16"/>
-<wire x1="32.41358125" y1="17.5" x2="29.90261875" y2="17.5" width="0.4572" layer="16"/>
-<wire x1="33.166421875" y1="16.747159375" x2="32.41358125" y2="17.5" width="0.4572" layer="16"/>
+<wire x1="32.41358125" y1="17.5" x2="31.10261875" y2="17.5" width="0.4572" layer="16"/>
+<wire x1="33.366421875" y1="16.547159375" x2="32.41358125" y2="17.5" width="0.4572" layer="16"/>
 </signal>
 <signal name="S$1">
 <contactref element="U$1" pad="1"/>
-<wire x1="30.751621875" y1="25.141959375" x2="30.851621875" y2="25.241959375" width="0.4572" layer="16"/>
+<wire x1="31.201621875" y1="25.141959375" x2="31.301621875" y2="25.241959375" width="0.4572" layer="16"/>
 </signal>
 <signal name="N$1">
@@
 <wire x1="8.541621875" y1="8.636959375" x2="9.604571875" y2="9.699909375" width="0.4572" layer="16"/>
 <wire x1="9.604571875" y1="9.699909375" x2="24.779571875" y2="9.699909375" width="0.4572" layer="16"/>
-<wire x1="25.9" y1="10.8203375" x2="25.9" y2="17.8" width="0.4572" layer="16"/>
-<wire x1="25.9" y1="17.8" x2="28.1" y2="20" width="0.4572" layer="16"/>
-<wire x1="24.779571875" y1="9.699909375" x2="25.9" y2="10.8203375" width="0.4572" layer="16"/>
+<wire x1="25.5" y1="10.4203375" x2="25.5" y2="17.4" width="0.4572" layer="16"/>
+<wire x1="25.5" y1="17.4" x2="28.1" y2="20" width="0.4572" layer="16"/>
+<wire x1="24.779571875" y1="9.699909375" x2="25.5" y2="10.4203375" width="0.4572" layer="16"/>
 <wire x1="28.1" y1="20" x2="30.9" y2="20" width="0.4572" layer="16"/>
 </signal>
@@
 <via x="13.783221875" y="4.164359375" extent="1-16" drill="0.85" diameter="1.8"/>
 <via x="22.346421875" y="7.117159375" extent="1-16" drill="0.85" diameter="1.8"/>
-<wire x1="27.6" y1="10.2707375" x2="24.446421875" y2="7.117159375" width="0.4572" layer="16"/>
+<wire x1="27.1" y1="9.7707375" x2="24.446421875" y2="7.117159375" width="0.4572" layer="16"/>
 <wire x1="22.346421875" y1="7.117159375" x2="24.446421875" y2="7.117159375" width="0.4572" layer="16"/>
-<wire x1="27.6" y1="10.2707375" x2="27.6" y2="17.4" width="0.4572" layer="16"/>
-<wire x1="32.50160625" y1="18.8" x2="33.10160625" y2="19.4" width="0.4572" layer="16"/>
-<wire x1="33.10160625" y1="22.19839375" x2="32.7" y2="22.6" width="0.4572" layer="16"/>
+<wire x1="27.1" y1="9.7707375" x2="27.1" y2="16.9" width="0.4572" layer="16"/>
+<wire x1="32.50160625" y1="18.8" x2="33.30160625" y2="19.6" width="0.4572" layer="16"/>
+<wire x1="33.30160625" y1="21.99839375" x2="32.7" y2="22.6" width="0.4572" layer="16"/>
 <wire x1="32.7" y1="22.6" x2="30.60261875" y2="22.6" width="0.4572" layer="16"/>
-<wire x1="27.6" y1="17.4" x2="29" y2="18.8" width="0.4572" layer="16"/>
+<wire x1="27.1" y1="16.9" x2="29" y2="18.8" width="0.4572" layer="16"/>
 <wire x1="29" y1="18.8" x2="32.50160625" y2="18.8" width="0.4572" layer="16"/>
-<wire x1="33.10160625" y1="19.4" x2="33.10160625" y2="22.19839375" width="0.4572" layer="16"/>
+<wire x1="33.30160625" y1="19.6" x2="33.30160625" y2="21.99839375" width="0.4572" layer="16"/>
 </signal>
 <signal name="N$5">
@@
 <signal name="GND">
 <wire x1="25.6723" y1="4.324303125" x2="25.6723" y2="6.146178125" width="0.4572" layer="16"/>
-<wire x1="28.8" y1="11.8" x2="29.4" y2="12.4" width="0.4572" layer="16"/>
-<wire x1="29.4" y1="12.4" x2="30.9" y2="12.4" width="0.4572" layer="16"/>
-<wire x1="25.6723" y1="6.146178125" x2="28.8" y2="9.273878125" width="0.4572" layer="16"/>
-<wire x1="28.8" y1="9.273878125" x2="28.8" y2="11.8" width="0.4572" layer="16"/>
+<wire x1="28.7" y1="11.3" x2="29.8" y2="12.4" width="0.4572" layer="16"/>
+<wire x1="29.8" y1="12.4" x2="30.9" y2="12.4" width="0.4572" layer="16"/>
+<wire x1="25.6723" y1="6.146178125" x2="28.7" y2="9.173878125" width="0.4572" layer="16"/>
+<wire x1="28.7" y1="9.173878125" x2="28.7" y2="11.3" width="0.4572" layer="16"/>
 </signal>
 </signals>
