File: Solar Cell/SolarCell.brd (EAGLE design)
At the start: 400 x 250 mm, 0 parts

Commit message: solar cell push
Parts:
- added E$1: (no value), Headers:61300211121
Routing:
- net S$1: track 1835.1 -> 330.4 mm
- net S$2: track 1207.8 -> 232.8 mm
- net S$4: track 193.0 -> 0.00 mm
- net S$3: track 195.6 -> 85.9 mm
- net S$9: track 0.00 -> 85.9 mm
- net S$28: track 0.00 -> 85.9 mm
- net S$26: track 0.00 -> 85.9 mm
- net S$24: track 0.00 -> 85.9 mm
- net S$22: track 0.00 -> 85.9 mm
- net S$20: track 0.00 -> 85.9 mm
- net S$18: track 0.00 -> 85.9 mm
- net S$16: track 0.00 -> 85.9 mm
- net S$14: track 0.00 -> 85.9 mm
- net S$12: track 0.00 -> 85.9 mm
- net S$8: track 0.00 -> 85.2 mm
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Other:
- board size 400 x 250 mm -> 119.4 x 96.5 mm
Changed lines of the file:
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@@
 <setting verticaltext="up"/>
 </settings>
-<grid distance="50" unitdist="mil" unit="mil" style="lines" multiple="1" display="no" altdistance="5" altunitdist="mil" altunit="mil"/>
+<grid distance="1" unitdist="mic" unit="mic" style="lines" multiple="1" display="no" altdistance="5" altunitdist="mil" altunit="mil"/>
 <layers>
 <layer number="1" name="Top" color="4" fill="1" visible="yes" active="yes"/>
@@
 <layer number="51" name="tDocu" color="7" fill="1" visible="yes" active="yes"/>
 <layer number="52" name="bDocu" color="7" fill="1" visible="yes" active="yes"/>
+<layer number="88" name="SimResults" color="9" fill="1" visible="no" active="no"/>
+<layer number="89" name="SimProbes" color="9" fill="1" visible="no" active="no"/>
+<layer number="90" name="Modules" color="5" fill="1" visible="no" active="no"/>
+<layer number="91" name="Nets" color="2" fill="1" visible="no" active="no"/>
+<layer number="92" name="Busses" color="1" fill="1" visible="no" active="no"/>
+<layer number="93" name="Pins" color="2" fill="1" visible="no" active="no"/>
+<layer number="94" name="Symbols" color="4" fill="1" visible="no" active="no"/>
+<layer number="95" name="Names" color="7" fill="1" visible="no" active="no"/>
+<layer number="96" name="Values" color="7" fill="1" visible="no" active="no"/>
+<layer number="97" name="Info" color="7" fill="1" visible="no" active="no"/>
+<layer number="98" name="Guide" color="6" fill="1" visible="no" active="no"/>
 </layers>
 <board>
 <plain>
-<wire x1="400" y1="228.41" x2="400" y2="21.59" width="0.1524" layer="20"/>
-<wire x1="400" y1="21.59" x2="378.41" y2="0" width="0.1524" layer="20" curve="-90"/>
-<wire x1="378.41" y1="0" x2="21.59" y2="0" width="0.1524" layer="20"/>
-<wire x1="21.59" y1="0" x2="0" y2="21.59" width="0.1524" layer="20" curve="-90"/>
-<wire x1="0" y1="21.59" x2="0" y2="228.41" width="0.1524" layer="20"/>
-<wire x1="0" y1="228.41" x2="21.59" y2="250" width="0.1524" layer="20" curve="-90"/>
-<wire x1="21.59" y1="250" x2="378.41" y2="250" width="0.1524" layer="20"/>
-<wire x1="378.41" y1="250" x2="400" y2="228.41" width="0.1524" layer="20" curve="-90"/>
+<wire x1="115.57" y1="1.27" x2="6.35" y2="1.27" width="0.1524" layer="20"/>
+<wire x1="6.35" y1="1.27" x2="1.27" y2="6.35" width="0.1524" layer="20" curve="-90"/>
+<wire x1="1.27" y1="6.35" x2="1.27" y2="92.71" width="0.1524" layer="20"/>
+<wire x1="1.27" y1="92.71" x2="6.35" y2="97.79" width="0.1524" layer="20" curve="-90"/>
+<wire x1="6.35" y1="97.79" x2="115.57" y2="97.79" width="0.1524" layer="20"/>
+<wire x1="115.57" y1="97.79" x2="120.65" y2="92.71" width="0.1524" layer="20" curve="-90"/>
+<wire x1="120.65" y1="92.71" x2="120.65" y2="6.35" width="0.1524" layer="20"/>
+<wire x1="120.65" y1="6.35" x2="115.57" y2="1.27" width="0.1524" layer="20" curve="-90"/>
 </plain>
 <attributes>
@@
 </autorouter>
 <elements>
+<element name="E$1" library="Headers" library_urn="urn:adsk.eagle:library:11687645" package="61300211121" package3d_urn="urn:adsk.eagle:package:11390690/2" value="" x="5.151" y="48.79" smashed="yes" rot="R90">
+<attribute name="NAME" x="2.992" y="45.488" size="1.27" layer="25" rot="R90"/>
+<attribute name="VALUE" x="8.834" y="45.488" size="1.27" layer="27" rot="R90"/>
+</element>
 </elements>
 <signals>
 <signal name="S$1">
-<wire x1="16.51" y1="139.7" x2="16.51" y2="234.95" width="13.97" layer="1"/>
-<wire x1="16.51" y1="234.95" x2="57.15" y2="234.95" width="13.97" layer="1"/>
-<wire x1="57.15" y1="234.95" x2="110.49" y2="234.95" width="13.97" layer="1"/>
-<wire x1="110.49" y1="234.95" x2="165.1" y2="234.95" width="13.97" layer="1"/>
-<wire x1="165.1" y1="234.95" x2="220.98" y2="234.95" width="13.97" layer="1"/>
-<wire x1="220.98" y1="234.95" x2="276.86" y2="234.95" width="13.97" layer="1"/>
-<wire x1="276.86" y1="234.95" x2="332.74" y2="234.95" width="13.97" layer="1"/>
-<wire x1="332.74" y1="234.95" x2="386.08" y2="234.95" width="13.97" layer="1"/>
-<wire x1="386.08" y1="234.95" x2="386.08" y2="13.97" width="13.97" layer="1"/>
-<wire x1="332.74" y1="234.95" x2="332.74" y2="40.64" width="13.97" layer="1"/>
-<wire x1="276.86" y1="234.95" x2="276.86" y2="43.18" width="13.97" layer="1"/>
-<wire x1="220.98" y1="234.95" x2="220.98" y2="45.72" width="13.97" layer="1"/>
-<wire x1="165.1" y1="234.95" x2="165.1" y2="44.45" width="13.97" layer="1"/>
-<wire x1="110.49" y1="234.95" x2="110.49" y2="43.18" width="13.97" layer="1"/>
-<wire x1="57.15" y1="234.95" x2="57.15" y2="43.18" width="13.97" layer="1"/>
+<wire x1="117.278" y1="94.604" x2="108.379" y2="94.604" width="2.2" layer="1"/>
+<wire x1="108.379" y1="94.604" x2="8.72" y2="94.604" width="2.2" layer="1"/>
+<wire x1="117.278" y1="94.604" x2="117.278" y2="4.454" width="2.2" layer="1"/>
+<wire x1="8.72" y1="94.604" x2="5.271" y2="91.155" width="2.2" layer="1"/>
+<wire x1="5.271" y1="91.155" x2="5.271" y2="50.238" width="2.2" layer="1"/>
+<wire x1="108.379" y1="94.604" x2="108.379" y2="8.73" width="2.2" layer="1"/>
 </signal>
 <signal name="S$2">
-<wire x1="17.78" y1="104.14" x2="17.78" y2="13.97" width="13.97" layer="1"/>
-<wire x1="17.78" y1="13.97" x2="83.82" y2="13.97" width="13.97" layer="1"/>
-<wire x1="83.82" y1="13.97" x2="138.43" y2="13.97" width="13.97" layer="1"/>
-<wire x1="138.43" y1="13.97" x2="193.04" y2="13.97" width="13.97" layer="1"/>
-<wire x1="193.04" y1="13.97" x2="248.92" y2="13.97" width="13.97" layer="1"/>
-<wire x1="248.92" y1="13.97" x2="356.87" y2="13.97" width="13.97" layer="1"/>
-<wire x1="248.92" y1="13.97" x2="248.92" y2="209.55" width="13.97" layer="1"/>
-<wire x1="193.04" y1="13.97" x2="193.04" y2="207.01" width="13.97" layer="1"/>
-<wire x1="138.43" y1="13.97" x2="138.43" y2="208.28" width="13.97" layer="1"/>
-<wire x1="83.82" y1="13.97" x2="83.82" y2="209.55" width="13.97" layer="1"/>
+<wire x1="9.105" y1="4.811" x2="112.829" y2="4.811" width="2.2" layer="1"/>
+<wire x1="112.829" y1="4.811" x2="112.829" y2="89.971" width="2.2" layer="1"/>
+<wire x1="9.105" y1="4.811" x2="5.24" y2="8.676" width="2.2" layer="1"/>
+<wire x1="5.24" y1="8.676" x2="5.24" y2="47.137" width="2.2" layer="1"/>
 </signal>
 <signal name="S$3">
-<wire x1="359.41" y1="13.97" x2="359.41" y2="209.55" width="13.97" layer="1"/>
-</signal>
-<signal name="S$4">
-<wire x1="304.8" y1="15.24" x2="304.8" y2="208.28" width="13.97" layer="1"/>
-</signal>
-<signal name="S$5">
-<wire x1="36.83" y1="104.14" x2="36.83" y2="96.52" width="2.54" layer="1"/>
-</signal>
-<signal name="S$6">
-<wire x1="33.02" y1="100.33" x2="40.64" y2="100.33" width="2.54" layer="1"/>
-</signal>
-<signal name="S$7">
-<wire x1="36.83" y1="144.78" x2="36.83" y2="137.16" width="2.54" layer="1"/>
+<wire x1="99.481" y1="94.426" x2="99.481" y2="8.552" width="2.2" layer="1"/>
+</signal>
+<signal name="S$8">
+<wire x1="103.931" y1="4.633" x2="103.931" y2="89.793" width="2.2" layer="1"/>
+</signal>
+<signal name="S$9">
+<wire x1="90.76" y1="94.426" x2="90.76" y2="8.552" width="2.2" layer="1"/>
+</signal>
+<signal name="S$10">
+<wire x1="95.21" y1="4.633" x2="95.21" y2="89.793" width="2.2" layer="1"/>
+</signal>
+<signal name="S$12">
+<wire x1="82.04" y1="94.426" x2="82.04" y2="8.552" width="2.2" layer="1"/>
+</signal>
+<signal name="S$13">
+<wire x1="86.49" y1="4.633" x2="86.49" y2="89.793" width="2.2" layer="1"/>
+</signal>
+<signal name="S$14">
+<wire x1="72.964" y1="94.247" x2="72.964" y2="8.373" width="2.2" layer="1"/>
+</signal>
+<signal name="S$15">
+<wire x1="77.414" y1="4.454" x2="77.414" y2="89.614" width="2.2" layer="1"/>
+</signal>
+<signal name="S$16">
+<wire x1="63.888" y1="94.782" x2="63.888" y2="8.908" width="2.2" layer="1"/>
+</signal>
+<signal name="S$17">
+<wire x1="68.338" y1="4.989" x2="68.338" y2="90.149" width="2.2" layer="1"/>
+</signal>
+<signal name="S$18">
+<wire x1="54.634" y1="94.782" x2="54.634" y2="8.908" width="2.2" layer="1"/>
+</signal>
+<signal name="S$19">
+<wire x1="59.084" y1="4.989" x2="59.084" y2="90.149" width="2.2" layer="1"/>
+</signal>
+<signal name="S$20">
+<wire x1="45.736" y1="94.604" x2="45.736" y2="8.73" width="2.2" layer="1"/>
+</signal>
+<signal name="S$21">
+<wire x1="50.186" y1="4.811" x2="50.186" y2="89.971" width="2.2" layer="1"/>
+</signal>
+<signal name="S$22">
+<wire x1="36.837" y1="94.782" x2="36.837" y2="8.908" width="2.2" layer="1"/>
+</signal>
+<signal name="S$23">
+<wire x1="41.287" y1="4.989" x2="41.287" y2="90.149" width="2.2" layer="1"/>
+</signal>
+<signal name="S$24">
+<wire x1="27.939" y1="94.782" x2="27.939" y2="8.908" width="2.2" layer="1"/>
+</signal>
+<signal name="S$25">
+<wire x1="32.389" y1="4.989" x2="32.389" y2="90.149" width="2.2" layer="1"/>
+</signal>
+<signal name="S$26">
+<wire x1="19.041" y1="94.96" x2="19.041" y2="9.086" width="2.2" layer="1"/>
+</signal>
+<signal name="S$27">
+<wire x1="23.491" y1="5.167" x2="23.491" y2="90.327" width="2.2" layer="1"/>
+</signal>
+<signal name="S$28">
+<wire x1="10.291" y1="94.96" x2="10.291" y2="9.086" width="2.2" layer="1"/>
+</signal>
+<signal name="S$29">
+<wire x1="14.741" y1="5.167" x2="14.741" y2="90.327" width="2.2" layer="1"/>
 </signal>
 </signals>
@@
 </board>
 </drawing>
+<compatibility>
+<note version="8.2" severity="warning">
+Since Version 8.2, EAGLE supports online libraries. The ids
+of those online libraries will not be understood (or retained)
+with this version.
+</note>
+<note version="8.3" severity="warning">
+Since Version 8.3, EAGLE supports URNs for individual library
+assets (packages, symbols, and devices). The URNs of those assets
+will not be understood (or retained) with this version.
+</note>
+<note version="8.3" severity="warning">
+Since Version 8.3, EAGLE supports the association of 3D packages
+with devices in libraries, schematics, and board files. Those 3D
+packages will not be understood (or retained) with this version.
+</note>
+</compatibility>
 </eagle>
